File: schematic/rak4260-soil-humidity/rak4260-soil-humidity.sch (KiCad schematic (older format))
At the start: 6 parts

Commit message: add settle time before measurement use d6 as sensor switch
Connections:
- net Moisture is gone; now on net A2: J?.3 (Pin_3)
- net Temp is gone; now on net A1: J?.2 (Pin_2)
- net D3: no longer R?.2
- net D6: now also R?.2
Other:
- note added: "green - temp"
- note added: "yellow - moisture"
- note removed: "green"
- note removed: "yellow"
Changed lines of the file:
@@
 	4850 2150 4900 2150
 Text Label 3950 2350 0    50   ~ 0
-D3
+D6
 Wire Wire Line
 	3950 2350 4100 2350
@@
 	5100 1500 4900 1500
 Text Label 5150 1600 0    50   ~ 0
-Temp
+A1
 Text Label 5150 1700 0    50   ~ 0
-Moisture
+A2
 Wire Wire Line
 	5150 1600 4900 1600
@@
 brown
 Text Notes 4600 1600 2    50   ~ 0
-green
+green - temp
 Text Notes 4600 1700 2    50   ~ 0
-yellow
+yellow - moisture
 Text Notes 4550 1800 2    50   ~ 0
 white
